Commit message: Support STVL on ROS2 Eloquent

File: neuronbot2_description/urdf/neuronbot2.urdf (robot description, URDF)
Before this commit: robot neuronbot2_description, 6 links, 5 joints
Links:
- added link camera_depth_optical_frame
- added link camera_rgb_frame
- added link camera_rgb_optical_frame
- added link realsense_depth_frame
- added link realsense_link; collision box size=0.012 0.132 0.020; visual mesh filename=package://turtlebot3_description/meshes/sensors/r200.dae
Joints:
- added joint camera_depth_optical_joint: type fixed, parent realsense_depth_frame, child camera_depth_optical_frame, origin xyz=0 0 0 rpy=-1.57 0 -1.57
- added joint camera_joint: type fixed, parent base_link, child realsense_link, origin xyz=0.1 0.0 0.1 rpy=0 0 0
- added joint camera_rgb_joint: type fixed, parent realsense_link, child camera_rgb_frame, origin xyz=0.005 0.018 0.013 rpy=-1.57 0 -1.57
- added joint camera_rgb_optical_joint: type fixed, parent camera_rgb_frame, child camera_rgb_optical_frame, origin xyz=0 0 0 rpy=-1.57 0 -1.57
- added joint realsense_depth_joint: type fixed, parent realsense_link, child realsense_depth_frame, origin xyz=0.005 0.028 0.013 rpy=-1.57 0 -1.57
